Commit message: fix xacro for sb modelc

File: xacro/modelc.xacro (robot description, xacro)
@@ -165,7 +165,25 @@
     <joint name="imu_joint" type="fixed">
         <axis xyz="0 1 0" />
-        <origin xyz="0.02 0 0.05" rpy="0 0.85521133347 3.14159265359"/>
+        <origin xyz="0.1 0 0.34" rpy="0 0 0"/>
         <parent link="base_link"/>
         <child link="imu"/>
+    </joint>
+    <!-- Livox Lidar -->
+    <link name="livox_frame">
+    </link>
+    <joint name="livox_joint" type="fixed">
+        <axis xyz="0 1 0" />
+        <origin xyz="0.2 0.0 0.175" rpy="0 0 0"/>
+        <parent link="base_link"/>
+        <child link="livox_frame"/>
+    </joint>
+    <!-- hikrobot_camera -->
+    <link name="hikrobot_camera">
+    </link>
+    <joint name="camera_joint" type="fixed">
+        <axis xyz="0 1 0" />
+        <origin xyz="0.3 0.0 0.35" rpy="0 0 0"/>
+        <parent link="base_link"/>
+        <child link="hikrobot_camera"/>
     </joint>
     <!-- ===============  Transmission =============== -->

Commit message: fix xacro
* xacroの修正
* display.launch用にrvizのConfig追加

File: xacro/modelc.xacro (robot description, xacro)
@@ -166,5 +166,5 @@
         <axis xyz="0 1 0" />
         <origin xyz="0.1 0 0.34" rpy="0 0 0"/>
-        <parent link="base_link"/>
+        <parent link="base_floor"/>
         <child link="imu"/>
     </joint>
@@ -175,5 +175,5 @@
         <axis xyz="0 1 0" />
         <origin xyz="0.2 0.0 0.175" rpy="0 0 0"/>
-        <parent link="base_link"/>
+        <parent link="base_floor"/>
         <child link="livox_frame"/>
     </joint>
@@ -184,5 +184,5 @@
         <axis xyz="0 1 0" />
         <origin xyz="0.3 0.0 0.35" rpy="0 0 0"/>
-        <parent link="base_link"/>
+        <parent link="base_floor"/>
         <child link="hikrobot_camera"/>
     </joint>

Commit message: Update xacro for mid 360

File: xacro/modelc.xacro (robot description, xacro)
@@ -1,246 +1,229 @@
 <?xml version="1.0"?>
-<robot xmlns:xacro="http://www.ros.org/wiki/xacro" name="whill_modelc" >
-    <link name="base_link">
+<robot xmlns:xacro="http://www.ros.org/wiki/xacro" name="whill_modelc">
+  <link name="base_link">
     </link>
-    <link name="base_floor">
-        <visual>
-            <geometry>
-                <box size="0.600 0.400 0.050"/>
-            </geometry>
-            <material name="grey">
-                <color rgba="0.5 0.5 0.5 1.0"/>
-            </material>
-        </visual>
-        <collision>
-            <geometry>
-                <box size="0.600 0.400 0.050"/>
-            </geometry>
-        </collision>
-        <inertial>
-            <origin xyz="0 0 0" rpy="0 0 0" />
-            <mass value="40" />
-            <inertia ixx="1.0"  ixy="0.0"   ixz="0.0"
-                                iyy="1.0"   iyz="0.0"
-                                            izz="1.0" />
-        </inertial>
+  <link name="base_floor">
+    <visual>
+      <geometry>
+        <box size="0.600 0.400 0.050"/>
+      </geometry>
+      <material name="grey">
+        <color rgba="0.5 0.5 0.5 1.0"/>
+      </material>
+    </visual>
+    <collision>
+      <geometry>
+        <box size="0.600 0.400 0.050"/>
+      </geometry>
+    </collision>
+    <inertial>
+      <origin xyz="0 0 0" rpy="0 0 0"/>
+      <mass value="40"/>
+      <inertia ixx="1.0" ixy="0.0" ixz="0.0" iyy="1.0" iyz="0.0" izz="1.0"/>
+    </inertial>
+  </link>
+  <joint name="base_body_joint" type="fixed">
+    <parent link="base_link"/>
+    <child link="base_floor"/>
+    <origin xyz="0.3 0 0.0" rpy="0 0 0"/>
+  </joint>
+  <link name="footrest_link">
+    <collision>
+      <geometry>
+        <box size="0.250 0.260 0.050"/>
+      </geometry>
+    </collision>
+    <visual>
+      <geometry>
+        <box size="0.250 0.260 0.050"/>
+      </geometry>
+      <material name="grey">
+        <color rgba="0.5 0.5 0.5 1.0"/>
+      </material>
+    </visual>
+    <inertial>
+      <origin xyz="0 0 0" rpy="0 0 0"/>
+      <mass value="1"/>
+      <inertia ixx="1.0" ixy="0.0" ixz="0.0" iyy="1.0" iyz="0.0" izz="1.0"/>
+    </inertial>
+  </link>
+  <joint name="footrest_joint" type="fixed">
+    <parent link="base_floor"/>
+    <child link="footrest_link"/>
+    <origin xyz="0.320 0 0" rpy="0 0 0"/>
+  </joint>
+  <link name="left_wheel_link">
+    <visual>
+      <geometry>
+        <cylinder length="0.05" radius="0.1325"/>
+      </geometry>
+      <origin xyz="0 0 0" rpy="0 0 0"/>
+      <material name="black"/>
+    </visual>
+    <collision>
+      <geometry>
+        <cylinder length="0.05" radius="0.1325"/>
+      </geometry>
+    </collision>
+    <inertial>
+      <origin xyz="0 0 0"/>
+      <mass value="0.500"/>
+      <inertia ixx="0.0013541667" ixy="0" ixz="0" iyy="0.0013541667" iyz="0" izz="0.0025"/>
+    </inertial>
+  </link>
+  <joint name="leftWheel" type="continuous">
+    <parent link="base_floor"/>
+    <child link="left_wheel_link"/>
+    <origin xyz="-0.3 0.245 0" rpy="-1.57 0 0"/>
+    <axis xyz="0 0 1"/>
+  </joint>
+  <link name="right_wheel_link">
+    <collision>
+      <origin xyz="0 0 0" rpy="0 0 0"/>
+      <geometry>
+        <cylinder length="0.05" radius="0.1325"/>
+      </geometry>
+    </collision>
+    <visual>
+      <origin xyz="0 0 0" rpy="0 0 0"/>
+      <geometry>
+        <cylinder length="0.05" radius="0.1325"/>
+      </geometry>
+      <material name="black"/>
+    </visual>
+    <inertial>
+      <origin xyz="0 0 0"/>
+      <mass value="0.500"/>
+      <inertia ixx="0.0013541667" ixy="0" ixz="0" iyy="0.0013541667" iyz="0" izz="0.0025"/>
+    </inertial>
+  </link>
+  <joint name="rightWheel" type="continuous">
+    <parent link="base_floor"/>
+    <child link="right_wheel_link"/>
+    <origin xyz="-0.3 -0.245 0" rpy="1.57 0 0"/>
+    <axis xyz="0 0 1"/>
+  </joint>
+  <link name="frontwheel_left">
+    <collision>
+      <geometry>
+        <cylinder length="0.05" radius="0.1325"/>
+      </geometry>
+    </collision>
+    <visual>
+      <geometry>
+        <cylinder length="0.05" radius="0.1325"/>
+      </geometry>
+      <material name="black"/>
+    </visual>
+    <inertial>
+      <origin xyz="0 0 0" rpy="0 0 0"/>
+      <mass value="1.0"/>
+      <inertia ixx="1.0" ixy="0.0" ixz="0.0" iyy="1.0" iyz="0.0" izz="1.0"/>
+    </inertial>
+  </link>
+  <joint name="frontwheel_left_joint" type="fixed">
+    <parent link="base_floor"/>
+    <child link="frontwheel_left"/>
+    <origin xyz="0.3 -0.245 0" rpy="1.57 0 0"/>
+    <axis xyz="0 0 1"/>
+  </joint>
+  <link name="frontwheel_right">
+    <collision>
+      <geometry>
+        <cylinder length="0.05" radius="0.1325"/>
+      </geometry>
+    </collision>
+    <visual>
+      <geometry>
+        <cylinder length="0.05" radius="0.1325"/>
+      </geometry>
+      <material name="black"/>
+    </visual>
+    <inertial>
+      <origin xyz="0 0 0" rpy="0 0 0"/>
+      <mass value="1.0"/>
+      <inertia ixx="1.0" ixy="0.0" ixz="0.0" iyy="1.0" iyz="0.0" izz="1.0"/>
+    </inertial>
+  </link>
+  <joint name="frontwheel_right_joint" type="fixed">
+    <parent link="base_floor"/>
+    <child link="frontwheel_right"/>
+    <origin xyz="0.3 0.245 0" rpy="1.57 0 0"/>
+    <axis xyz="0 0 -1"/>
+  </joint>
+  <!-- IMU -->
+  <link name="imu">
     </link>
-    <joint name="base_body_joint" type="fixed">
-        <parent link="base_link" />
-        <child link="base_floor" />
-        <origin xyz="0.3 0 0.0" rpy="0 0 0"/>
+  <joint name="imu_joint" type="fixed">
+    <axis xyz="0 1 0"/>
+    <origin xyz="0.1 0 0.34" rpy="0 0 0"/>
+    <parent link="base_floor"/>
+    <child link="imu"/>
+  </joint>
+  <!-- Livox Lidar -->
+  <link name="livox_frame">
+    </link>
+  <joint name="livox_joint" type="fixed">
+    <axis xyz="0 1 0"/>
+    <origin xyz="0.2 0.3 1.4" rpy="0 0 0"/>
+    <parent link="base_floor"/>
+    <child link="livox_frame"/>
+  </joint>
+  <!-- ===============  Transmission =============== -->
+  <transmission name="right_wheel_trans">
+    <type>transmission_interface/SimpleTransmission</type>
+    <joint name="rightWheel">
+      <hardwareInterface>hardware_interface/VelocityJointInterface</hardwareInterface>
     </joint>
-    <link name="footrest_link">
-        <collision>
-            <geometry>
-                <box size="0.250 0.260 0.050"/>
-            </geometry>
-        </collision>
-        <visual>
-            <geometry>
-                <box size="0.250 0.260 0.050"/>
-            </geometry>
-            <material name="grey">
-                <color rgba="0.5 0.5 0.5 1.0"/>
-            </material>
-        </visual>
-        <inertial>
-            <origin xyz="0 0 0" rpy="0 0 0" />
-            <mass value="1" />
-            <inertia ixx="1.0"  ixy="0.0"   ixz="0.0"
-                                iyy="1.0"   iyz="0.0"
-                                            izz="1.0" />
-        </inertial>
-    </link>
-    <joint name="footrest_joint" type="fixed">
-        <parent link="base_floor" />
-        <child link="footrest_link" />
-        <origin xyz="0.320 0 0" rpy="0 0 0"/>
+    <actuator name="right_wheel_motor">
+      <hardwareInterface>hardware_interface/VelocityJointInterface</hardwareInterface>
+      <mechanicalReduction>30</mechanicalReduction>
+    </actuator>
+  </transmission>
+  <transmission name="left_wheel_trans">
+    <type>transmission_interface/SimpleTransmission</type>
+    <joint name="leftWheel">
+      <hardwareInterface>hardware_interface/VelocityJointInterface</hardwareInterface>
     </joint>
-    <link name="left_wheel_link">
-        <visual>
-            <geometry>
-                <cylinder length="0.05" radius="0.1325"/>
-            </geometry>
-            <origin xyz="0 0 0" rpy="0 0 0" />
-            <material name="black" />
-        </visual>
-        <collision>
-            <geometry>
-                <cylinder length="0.05" radius="0.1325"/>
-            </geometry>
-        </collision>
-        <inertial>
-            <origin xyz="0 0 0"/>
-            <mass value="0.500"/>
-            <inertia ixx="0.0013541667" ixy="0" ixz="0" iyy="0.0013541667" iyz="0" izz="0.0025"/>
-        </inertial>
-    </link>
-    <joint name="leftWheel" type="continuous">
-        <parent link="base_floor" />
-        <child link="left_wheel_link" />
-        <origin xyz="-0.3 0.245 0" rpy="-1.57 0 0" />
-        <axis xyz="0 0 1" />
-    </joint>
-    <link name="right_wheel_link">
-        <collision>
-            <origin xyz="0 0 0" rpy="0 0 0" />
-            <geometry>
-                <cylinder length="0.05" radius="0.1325"/>
-            </geometry>
-        </collision>
-        <visual>
-            <origin xyz="0 0 0" rpy="0 0 0" />
-            <geometry>
-                <cylinder length="0.05" radius="0.1325"/>
-            </geometry>
-            <material name="black" />
-        </visual>
-        <inertial>
-            <origin xyz="0 0 0"/>
-            <mass value="0.500"/>
-            <inertia ixx="0.0013541667" ixy="0" ixz="0" iyy="0.0013541667" iyz="0" izz="0.0025"/>
-        </inertial>
-    </link>
-    <joint name="rightWheel" type="continuous">
-        <parent link="base_floor" />
-        <child link="right_wheel_link" />
-        <origin xyz="-0.3 -0.245 0" rpy="1.57 0 0" />
-        <axis xyz="0 0 1" />
-    </joint>
-    <link name="frontwheel_left">
-        <collision>
-            <geometry>
-                <cylinder length="0.05" radius="0.1325"/>
-            </geometry>
-        </collision>
-        <visual>
-            <geometry>
-                <cylinder length="0.05" radius="0.1325"/>
-            </geometry>
-            <material name="black" />
-        </visual>
-        <inertial>
-            <origin xyz="0 0 0" rpy="0 0 0" />
-            <mass value="1.0" />
-            <inertia ixx="1.0"  ixy="0.0"   ixz="0.0"
-                                iyy="1.0"   iyz="0.0"
-                                            izz="1.0" />
-        </inertial>
-    </link>
-    <joint name="frontwheel_left_joint" type="fixed">
-        <parent link="base_floor" />
-        <child link="frontwheel_left" />
-        <origin xyz="0.3 -0.245 0" rpy="1.57 0 0" />
-        <axis xyz="0 0 1" />
-    </joint>
-    <link name="frontwheel_right">
-        <collision>
-            <geometry>
-                <cylinder length="0.05" radius="0.1325"/>
-            </geometry>
-        </collision>
-        <visual>
-            <geometry>
-                <cylinder length="0.05" radius="0.1325"/>
-            </geometry>
-            <material name="black" />
-        </visual>
-        <inertial>
-            <origin xyz="0 0 0" rpy="0 0 0" />
-            <mass value="1.0" />
-            <inertia ixx="1.0"  ixy="0.0"   ixz="0.0"
-                                iyy="1.0"   iyz="0.0"
-                                            izz="1.0" />
-        </inertial>
-    </link>
-    <joint name="frontwheel_right_joint" type="fixed">
-        <parent link="base_floor" />
-        <child link="frontwheel_right"/>
-        <origin xyz="0.3 0.245 0" rpy="1.57 0 0" />
-        <axis xyz="0 0 -1" />
-    </joint>
-    <!-- IMU -->
-    <link name="imu">
-    </link>
-    <joint name="imu_joint" type="fixed">
-        <axis xyz="0 1 0" />
-        <origin xyz="0.1 0 0.34" rpy="0 0 0"/>
-        <parent link="base_floor"/>
-        <child link="imu"/>
-    </joint>
-    <!-- Livox Lidar -->
-    <link name="livox_frame">
-    </link>
-    <joint name="livox_joint" type="fixed">
-        <axis xyz="0 1 0" />
-        <origin xyz="0.2 0.0 0.175" rpy="0 0 0"/>
-        <parent link="base_floor"/>
-        <child link="livox_frame"/>
-    </joint>
-    <!-- hikrobot_camera -->
-    <link name="hikrobot_camera">
-    </link>
-    <joint name="camera_joint" type="fixed">
-        <axis xyz="0 1 0" />
-        <origin xyz="0.3 0.0 0.35" rpy="0 0 0"/>
-        <parent link="base_floor"/>
-        <child link="hikrobot_camera"/>
-    </joint>
-    <!-- ===============  Transmission =============== -->
-    <transmission name="right_wheel_trans">
-        <type>transmission_interface/SimpleTransmission</type>
-        <joint name="rightWheel">
-            <hardwareInterface>hardware_interface/VelocityJointInterface</hardwareInterface>
-        </joint>
-        <actuator name="right_wheel_motor">
-            <hardwareInterface>hardware_interface/VelocityJointInterface</hardwareInterface>
-            <mechanicalReduction>30</mechanicalReduction>
-        </actuator>
-    </transmission>
-    <transmission name="left_wheel_trans">
-        <type>transmission_interface/SimpleTransmission</type>
-        <joint name="leftWheel">
-            <hardwareInterface>hardware_interface/VelocityJointInterface</hardwareInterface>
-        </joint>
-        <actuator name="left_wheel_motor">
-            <hardwareInterface>hardware_interface/VelocityJointInterface</hardwareInterface>
-            <mechanicalReduction>30</mechanicalReduction>
-        </actuator>
-    </transmission>
-    <!-- For Gazebo -->
-    <gazebo>
-        <plugin name="gazebo_ros_control" filename="libgazebo_ros_control.so">
-            <robotNamespace>/whill_simulator</robotNamespace>
-        </plugin>
-    </gazebo>
-    <gazebo reference="base_floor">
-        <selfCollide>true</selfCollide>
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